File: pcb/Shapeshifter_4060_v2_3/kicad/Backup.kicad_pcb (KiCad board)
At the start: 2 copper layers, 285 x 94.6 mm, 117 parts, among them J1 Conn_01x16, J1 MINI, J2 Conn_01x12, SW1 TAB, SW10 O, SW11 P, SW12 BKSP, SW13 ESC, SW14 A, SW15 S, SW16 D, SW17 F/LOWER, SW18 G, SW19 H, SW2 Q, SW20 J/RAISE, SW21 K, SW22 L, SW23 ;, SW24 ", SW25 SHIFT, SW26 Z, SW27 X, SW28 C, SW29 V, SW3 W, SW30 B, SW31 N, SW32 M, SW33 ,, SW34 ., SW35 /, SW36 ENTER, SW37 HYPER, SW38 CTRL/GRV, SW39 ALT/TAB, SW4 E, SW40 CMD, SW41 BKSP/LIFT, SW42 SHIFT, SW43 SPACE, SW44 ENTER/LIFT, SW45 LEFT, SW46 DOWN, SW47 UP, SW48 RIGHT, SW49 SPECIAL, SW5 R, SW50 SPECIAL, SW6 T, SW7 Y, SW8 U, SW9 I, U1 AdafruitFeather32u4BLE

Commit message: update shapeshifter to use newer components from non-ble library, move mdbt40
Parts:
- removed D50: DIODE, Laptreus v2 Footprints:Diode-dual
- removed the FID at (94.7, 144.7)
- removed the FID at (373.1, 57.3)
- removed HOLE (x2): VAL**, hole:PKRHSL
- removed HOLE: VAL**, hole:PKRHC
- removed HOLE (x3): VAL**, hole:PKRH
- removed the J1 at (109.6, 53.7)
- removed the J1 at (223.9, 54.7)
- removed S0: DTSM-6, dtsm:KSEM31GLFS
- removed SW49, SW50: SPECIAL, Laptreus v2 Footprints:Hybrid_Kailh_MX_Socket_Through_Hole
- added C1: 10µF, Laptreus v2 Footprints:Capacitor-0805MP, F.Cu at (372.5, 93.7)
- added C2: 1µF, Laptreus v2 Footprints:Capacitor-0805MP, F.Cu at (238.4, 80.1)
- added C20: 100nF, Laptreus v2 Footprints:Capacitor-0805MP, F.Cu at (372.5, 83.2)
- added C3: 10µF, Laptreus v2 Footprints:Capacitor-0805MP, F.Cu at (372.5, 96.0)
- added C4: 1µF, Laptreus v2 Footprints:Capacitor-0805MP, F.Cu at (241.4, 132.8)
- added C5: 10µF, Laptreus v2 Footprints:Capacitor-0805MP, F.Cu at (254.6, 98.1)
- added C6: 1µF, Laptreus v2 Footprints:Capacitor-0805MP, F.Cu at (244.9, 124.9)
- added C7: 1µF, Laptreus v2 Footprints:Capacitor-0805MP, F.Cu at (232.9, 116.4)
- added F1: Polyfuse, Fuse_Holders_and_Fuses:Fuse_SMD1206_Reflow, F.Cu at (372.5, 86.2)
- added FID: FIDUCIAL, hole:FIDUCIAL, B.Cu at (372.7, 163.3)
- added FID: FIDUCIAL, hole:FIDUCIAL, B.Cu at (92.8, 74.0)
- added FID: FIDUCIAL, hole:FIDUCIAL, F.Cu at (92.8, 74.0)
- added FID: FIDUCIAL, hole:FIDUCIAL, F.Cu at (372.7, 163.3)
- added IC1: ATMEGA32U4, Package_QFP:TQFP-44_10x10mm_P0.8mm, F.Cu at (233.0, 128.3)
- added J1: HRO-TYPE-C-31-M-12, Laptreus v2 Footprints:HRO-TYPE-C-31-M-12, F.Cu at (357.4, 70.2)
- added JP1: PINHD-1X1CB, Adafruit NeoPixel Ring 12:1X01-CLEANBIG, F.Cu at (213.0, 124.5)
- added JP2: PINHD-1X1CB, Adafruit NeoPixel Ring 12:1X01-CLEANBIG, F.Cu at (213.0, 121.5)
- added JP3: PINHD-1X1CB, Adafruit NeoPixel Ring 12:1X01-CLEANBIG, F.Cu at (213.0, 127.5)
- added L1: YELLOW, Adafruit Feather 32u4 Bluefruit LE:CHIPLED_0805_NOOUTLINE, B.Cu at (229.6, 74.1)
- added L2: RED, Adafruit Feather 32u4 Bluefruit LE:CHIPLED_0805_NOOUTLINE, B.Cu at (233.9, 74.1)
- added L3: BLUE, Adafruit Feather 32u4 Bluefruit LE:CHIPLED_0805_NOOUTLINE, B.Cu at (238.0, 74.2)
- added L4: ORANGE, Adafruit Feather 32u4 Bluefruit LE:CHIPLED_0805_NOOUTLINE, B.Cu at (224.8, 74.1)
- added R10: 1K, Laptreus v2 Footprints:0805-NO, F.Cu at (237.1, 137.3)
- added R11: 5.1K, Laptreus v2 Footprints:0805-NO, F.Cu at (372.5, 73.2)
- added R12: 5.1K, Laptreus v2 Footprints:0805-NO, F.Cu at (372.5, 75.7)
- added R13: 2.2K, Laptreus v2 Footprints:0805-NO, F.Cu at (229.6, 74.0)
- added R3: 10K, Laptreus v2 Footprints:0805-NO, F.Cu at (248.9, 111.4)
- added R4: 100K, Laptreus v2 Footprints:0805-NO, F.Cu at (253.1, 115.5)
- added R5: 100K, Laptreus v2 Footprints:0805-NO, F.Cu at (253.1, 119.2)
- added R6: 2.2K, Laptreus v2 Footprints:0805-NO, F.Cu at (233.8, 74.0)
- added R7: 2.2K, Laptreus v2 Footprints:0805-NO, F.Cu at (238.0, 74.1)
- added R8: 22, Laptreus v2 Footprints:0805-NO, F.Cu at (372.5, 78.2)
- added R9: 22, Laptreus v2 Footprints:0805-NO, F.Cu at (372.5, 80.7)
- added S1: Screw, Laptreus v2 Footprints:PKRH-Round, F.Cu at (115.7, 99.4)
- added S2: Screw, Laptreus v2 Footprints:PKRH, F.Cu at (350.5, 99.4)
- added S3: Screw, Laptreus v2 Footprints:PKRH, F.Cu at (218.8, 118.7)
- added S4: Screw, Laptreus v2 Footprints:PKRHSL-NPTH, F.Cu at (92.5, 128.3)
- added S5: Screw, Laptreus v2 Footprints:PKRHSL-NPTH, F.Cu at (373.5, 128.3)
- added S6: Screw, Laptreus v2 Footprints:PKRH, F.Cu at (281.0, 156.7)
- added S7: Tofu screw, Laptreus v2 Footprints:PKRH, F.Cu at (233.0, 109.0)
- added S8: Tofu screw, Laptreus v2 Footprints:PKRH, F.Cu at (116.7, 156.9)
- added S9: Tofu screw, Laptreus v2 Footprints:PKRH, F.Cu at (350.5, 156.9)
- added SW_POW_EN2: SW_SPDT, Laptreus v2 Footprints:EG1218, B.Cu at (157.5, 132.7)
- added SW_RESET2: SWITCH_PUSH, Laptreus v2 Footprints:Hybrid_Kailh_MX_Socket_Through_Hole_No_Alignment_Pad, F.Cu at (233.1, 93.8)
- added TP1: SWCLK, Adafruit Feather 32u4 Bluefruit LE:PAD-1.5X2.0, B.Cu at (248.4, 82.1)
- added TP2: SWDIO, Adafruit Feather 32u4 Bluefruit LE:PAD-1.5X2.0, B.Cu at (248.4, 84.5)
- added TP3: SWDIO, Adafruit Feather 32u4 Bluefruit LE:PAD-1.5X2.0, B.Cu at (248.4, 86.9)
- added U2: SPX3819-3.3, Adafruit Feather 32u4 Bluefruit LE:SOT23-5, F.Cu at (372.5, 90.2)
- added U3: MDBT40, Adafruit Feather 32u4 Bluefruit LE:BLE_MODULE_RAYTAC_MDBT40, F.Cu at (247.0, 80.6)
- added U6: USBLC6-2SC6, Laptreus v2 Footprints:USBLC6-2SC6, F.Cu at (367.5, 79.5)
- added X1: JSTPH, Laptreus v2 Footprints:JSTPH2-with-THT, B.Cu at (259.3, 78.6)
- added X2: JSTPH, Laptreus v2 Footprints:JSTPH2-with-THT, F.Cu at (254.8, 127.2)
- added Y1: 8MHz, Adafruit Feather 32u4 Bluefruit LE:RESONATOR-SMD, F.Cu at (222.5, 127.9)
- D49: value DIODE -> MBR120; footprint Laptreus v2 Footprints:Diode-dual -> Adafruit Feather 32u4 Bluefruit LE:SOD-123
- J2: value Conn_01x12 -> ISP; footprint Connector_PinHeader_2.54mm:PinHeader_1x12_P2.54mm_Vertical -> Laptreus v2 Footprints:isp_standard; moved to B.Cu
- R1: value 22 -> 1K; footprint 0805:0805R -> Laptreus v2 Footprints:0805-NO; moved to F.Cu
- R2: value 22 -> 100K; footprint 0805:0805R -> Laptreus v2 Footprints:0805-NO; moved to F.Cu
- SW1: footprint Laptreus v2 Footprints:Hybrid_Kailh_MX_Socket_Through_Hole -> Laptreus v2 Footprints:Hybrid_Kailh_MX_Socket_No_Alignment_Pad
- SW10, SW11, SW12, SW13, SW14, SW15, SW16, SW17, SW18, SW19, SW2, SW20, SW21, SW22, SW23, SW24, SW25, SW26, SW27, SW28, SW29, SW3, SW30, SW31, SW32, SW33, SW34, SW35, SW36, SW37, SW38, SW39, SW4, SW40, SW45, SW46, SW47, SW48, SW5, SW6, SW7, SW8, SW9: footprint Laptreus v2 Footprints:Hybrid_Kailh_MX_Socket_Through_Hole -> Laptreus v2 Footprints:Hybrid_Kailh_MX_Socket_Through_Hole_No_Alignment_Pad
- SW41: value BKSP/LIFT -> SHIFT; footprint Laptreus v2 Footprints:Hybrid_Kailh_MX_Socket_Through_Hole -> Laptreus v2 Footprints:Hybrid_Kailh_MX_Socket_Through_Hole_No_Alignment_Pad
- SW42: value SHIFT -> BKSP/LIFT; footprint Laptreus v2 Footprints:Hybrid_Kailh_MX_Socket_Through_Hole -> Laptreus v2 Footprints:Hybrid_Kailh_MX_Socket_Through_Hole_No_Alignment_Pad
- SW43: value SPACE -> ENTER/LIFT; footprint Laptreus v2 Footprints:Hybrid_Kailh_MX_Socket_Through_Hole -> Laptreus v2 Footprints:Hybrid_Kailh_MX_Socket_Through_Hole_No_Alignment_Pad
- SW44: value ENTER/LIFT -> SPACE; footprint Laptreus v2 Footprints:Hybrid_Kailh_MX_Socket_Through_Hole -> Laptreus v2 Footprints:Hybrid_Kailh_MX_Socket_Through_Hole_No_Alignment_Pad
- SW_RESET1: moved to B.Cu
- U1: value AdafruitFeather32u4BLE -> MCP73831T-2ATI/OT; footprint Laptreus v2 Footprints:Adafruit Feather 32u4 BLE -> Adafruit Feather 32u4 Bluefruit LE:SOT23-5
- moved R2 257.5 mm to (367.5, 90.2), turned to 0 degrees
- moved R1 116.1 mm to (224.9, 74.1)
- moved D49 75.1 mm to (253.3, 104.1), turned to 90 degrees
- moved SW_RESET1 47.7 mm to (247.7, 95.7), turned to 0 degrees
- moved U1 34.6 mm to (243.9, 106.8), turned to 180 degrees
- moved SW41 27.4 mm to (270.0, 153.1), turned to 40 degrees
- moved SW44 26.5 mm to (196.0, 153.1), turned to 320 degrees
- moved D40 25.9 mm to (293.6, 157.2)
- moved D38 25.9 mm to (331.2, 150.6)
- moved D39 25.9 mm to (312.4, 153.9)
- moved D37 25.9 mm to (349.9, 147.2)
- moved SW37 25.8 mm to (348.4, 138.6)
- moved SW38 25.8 mm to (329.7, 142.0)
- moved SW39 25.8 mm to (310.9, 145.3)
- moved SW40 25.8 mm to (292.1, 148.6)
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Connections:
- D1 pad 2: /COL10 -> /COL11
- D12 pad 2: /COL4 -> /COL0
- D13 pad 2: /COL9 -> /COL11
- D24 pad 2: /COL3 -> /COL0
- D25 pad 2: /COL8 -> /COL11
- D36 pad 2: /COL2 -> /COL0
- D37 pad 2: /COL7 -> /COL11
- D48 pad 2: /COL1 -> /COL0
- J2 pad 1: /COL5 -> MISO
- J2 pad 2: /COL4 -> +3V3
- J2 pad 3: /COL6 -> SCK
- J2 pad 4: /COL7 -> MOSI
- J2 pad 5: Net-(J2-Pad5) -> RST
- J2 pad 6: /COL8 -> GND
- R1 pad 1: (no net) -> +5V
- R1 pad 2: (no net) -> /CHARGE
- R2 pad 1: (no net) -> +5V
- R2 pad 2: (no net) -> /EN
- SW1 pad 1: /ROW4 -> /ROW0
- SW12 pad 1: /ROW4 -> /ROW0
- SW13 pad 1: /ROW4 -> /ROW1
- SW24 pad 1: /ROW4 -> /ROW1
- SW25 pad 1: /ROW4 -> /ROW2
- SW36 pad 1: /ROW4 -> /ROW2
- SW37 pad 1: /ROW4 -> /ROW3
- SW48 pad 1: /ROW4 -> /ROW3
- SW_POW_EN1 pad 2: /Enable -> /EN
- SW_POW_EN1 pad 3: (no net) -> Net-(SW_POW_EN1-Pad3)
- U1 pad 1: (no net) -> Net-(L4-PadC)
- U1 pad 2: (no net) -> GND
- U1 pad 3: (no net) -> +3.7VBAT
- U1 pad 4: (no net) -> +5V
- U1 pad 5: (no net) -> Net-(R3-Pad1)
Routing:
- net /ROW0: track 0.00 -> 381.9 mm, vias 0 -> 2
- net /ROW1: track 0.00 -> 350.5 mm, vias 0 -> 6
- net /ROW2: track 0.00 -> 305.6 mm, vias 0 -> 6
- net /COL10: track 0.00 -> 297.7 mm, vias 0 -> 1
- net /ROW3: track 0.00 -> 292.8 mm, vias 0 -> 6
- net /COL11: track 0.00 -> 238.2 mm, vias 0 -> 1
- net /COL0: track 0.00 -> 224.2 mm, vias 0 -> 1
- net /EN: track 0.00 -> 209.2 mm, vias 0 -> 8
- net /COL1: track 0.00 -> 203.7 mm, vias 0 -> 1
- net /COL9: track 0.00 -> 201.2 mm, vias 0 -> 1
- net /COL2: track 0.00 -> 187.0 mm, vias 0 -> 1
- net /COL8: track 0.00 -> 185.3 mm, vias 0 -> 1
- net /COL3: track 0.00 -> 170.3 mm, vias 0 -> 1
- net /COL7: track 0.00 -> 157.6 mm, vias 0 -> 1
- net GND: track 0.00 -> 149.8 mm, vias 0 -> 35
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- added copper zone on F.Cu, net (none)
- added copper zone on B.Cu, net +3V3
Other:
- net class Default: trace_width 0.25 -> 0.2; via_dia 0.9 -> 0.6; via_drill 0.6 -> 0.4
- net class Ground: trace_width 0.4 -> 0.25
- net class Power: trace_width 0.4 -> 0.25
- net class USB added: clearance 0.2, trace_width 0.2, via_dia 0.6, via_drill 0.4
- rule trace_min: 0.25 -> 0.2
- rule via_min_drill: 0.6 -> 0.4
- rule via_min_size: 0.9 -> 0.6
- board text added: "+3V3"
- board text added: "1Ah (51x34x5.9)"
- board text added: "400mAh (27x37x5)"
- board text added: "B7"
- board text added: "ESD PROTECTION"
- board text added: "GND"
- board text added: "JLCJLCJLCJLC"
- board text added: "LiPo Charge Circuit"
- board text added: "NORDIC nRF52832 BLE MODULE"
- board text added: "Red - Mode Blue - Connected Yellow - Pin 13 Orange - Charging"
- board text added: "Schotky"
- board text added: "Voltage Regulator"
