File: pcb/Shapeshifter_4060_v2_3/kicad/Laptreus-v2.kicad_pcb (KiCad board)
At the start: 2 copper layers, 285 x 94.6 mm, 156 parts, among them IC1 ATMEGA32U4, J1 HRO-TYPE-C-31-M-12, J2 ISP, SW1 TAB, SW10 O, SW11 P, SW12 BKSP, SW13 ESC, SW14 A, SW15 S, SW16 D, SW17 F/LOWER, SW18 G, SW19 H, SW2 Q, SW20 J/RAISE, SW21 K, SW22 L, SW23 ;, SW24 ", SW25 SHIFT, SW26 Z, SW27 X, SW28 C, SW29 V, SW3 W, SW30 B, SW31 N, SW32 M, SW33 ,, SW34 ., SW35 /, SW36 ENTER, SW37 HYPER, SW38 CTRL/GRV, SW39 ALT/TAB, SW4 E, SW40 CMD, SW41 SHIFT, SW42 BKSP/LIFT, SW43 ENTER/LIFT, SW44 SPACE, SW45 LEFT, SW46 DOWN, SW47 UP, SW48 RIGHT, SW5 R, SW6 T, SW7 Y, SW8 U, SW9 I, U1 MCP73831T-2ATI/OT, U2 SPX3819-3.3, U3 MDBT40, U6 USBLC6-2SC6, X1 JSTPH, X2 JSTPH, Y1 8MHz

Commit message: update shapeshifter to use newer components from non-ble library, move mdbt40
Parts:
- removed S1: Screw, Laptreus v2 Footprints:PKRH-Round
- removed S2, S3, S6: Screw, Laptreus v2 Footprints:PKRH
- removed S4, S5: Screw, Laptreus v2 Footprints:PKRHSL-NPTH
- removed S7, S8: Tofu screw, Laptreus v2 Footprints:PKRH
- removed SW_RESET2: SWITCH_PUSH, Laptreus v2 Footprints:Hybrid_Kailh_MX_Socket_Through_Hole_No_Alignment_Pad
- removed TP1: SWCLK, Adafruit Feather 32u4 Bluefruit LE:PAD-1.5X2.0
- removed TP2, TP3: SWDIO, Adafruit Feather 32u4 Bluefruit LE:PAD-1.5X2.0
- added BOARD1: BoardOutline, Laptreus v2_2 Archive Footprints:60-percent-plus-tofu, F.Cu at (233.0, 118.9)
- added J3: Conn_ARM_JTAG_SWD_10, Connector_PinHeader_1.27mm:PinHeader_2x05_P1.27mm_Vertical, F.Cu at (121.0, 159.7)
- D1, D10, D11, D12, D13, D14, D15, D16, D17, D18, D19, D2, D20, D21, D22, D23, D24, D25, D26, D27, D28, D29, D3, D30, D31, D32, D33, D34, D35, D36, D37, D38, D39, D4, D40, D41, D42, D43, D44, D45, D46, D47, D48, D5, D6, D7, D8, D9: footprint Laptreus v2 Footprints:Diode-dual -> Laptreus v2_2 Archive Footprints:D_SOD-323_With_Adhesive
- F1: footprint Fuse_Holders_and_Fuses:Fuse_SMD1206_Reflow -> Laptreus v2_2 Archive Footprints:Fuse_1812_4532Metric_With_Adhesive
- FID1, FID2, FID3, FID4: renamed from FID; value FIDUCIAL -> Fiducial; footprint hole:FIDUCIAL -> Laptreus v2_2 Archive Footprints:FIDUCIAL
- IC1: footprint Package_QFP:TQFP-44_10x10mm_P0.8mm -> Laptreus v2_2 Archive Footprints:TQFP-44_10x10mm_P0.8mm
- L1, L2, L3, L4: footprint Adafruit Feather 32u4 Bluefruit LE:CHIPLED_0805_NOOUTLINE -> Laptreus v2_2 Archive Footprints:LED_0603_1608Metric_Castellated_With_Adhesive
- R1, R13, R6, R7: footprint Laptreus v2 Footprints:0805-NO -> Laptreus v2_2 Archive Footprints:R_0603_1608Metric_With_Adhesive; moved to B.Cu
- R10, R11, R12, R2, R3, R4, R5, R8, R9: footprint Laptreus v2 Footprints:0805-NO -> Laptreus v2_2 Archive Footprints:R_0603_1608Metric_With_Adhesive
- SW1: footprint Laptreus v2 Footprints:Hybrid_Kailh_MX_Socket_No_Alignment_Pad -> Laptreus v2_2 Archive Footprints:Hybrid_Kailh_MX_Choc_Socket_Through_Hole_With_Diode
- SW10, SW11, SW12, SW13, SW15, SW16, SW17, SW18, SW19, SW2, SW20, SW21, SW22, SW26, SW27, SW28, SW29, SW3, SW30, SW31, SW32, SW33, SW34, SW35, SW37, SW38, SW39, SW4, SW40, SW41, SW42, SW43, SW44, SW45, SW46, SW47, SW48, SW5, SW6, SW7, SW8, SW9: footprint Laptreus v2 Footprints:Hybrid_Kailh_MX_Socket_Through_Hole_No_Alignment_Pad -> Laptreus v2_2 Archive Footprints:Hybrid_Kailh_MX_Choc_Socket_Through_Hole_With_Diode
- SW14, SW23, SW24, SW25, SW36: footprint Laptreus v2 Footprints:Hybrid_Kailh_MX_Socket_Through_Hole_No_Alignment_Pad -> Laptreus v2_2 Archive Footprints:Hybrid_Kailh_MX_Choc_Socket_Through_Hole_With_Diode_No_Diode_Trace
- U1, U2: footprint Adafruit Feather 32u4 Bluefruit LE:SOT23-5 -> Laptreus v2_2 Archive Footprints:SOT-143_With_Adhesive
- U3: moved to B.Cu
- X1, X2: footprint Laptreus v2 Footprints:JSTPH2-with-THT -> Laptreus v2_2 Archive Footprints:JSTPH2-with-THT
- moved L3 163.3 mm to (94.5, 152.2)
- moved U3 162.3 mm to (103.8, 157.0)
- moved L2 161.1 mm to (94.5, 155.0)
- moved R7 159.4 mm to (94.4, 143.5), turned to 0 degrees
- moved L1 158.9 mm to (94.5, 157.7)
- moved R6 156.6 mm to (94.5, 145.5), turned to 0 degrees
- moved L4 156.4 mm to (94.5, 160.5)
- moved R13 153.8 mm to (94.5, 147.5), turned to 180 degrees
- moved R1 150.6 mm to (94.4, 149.4), turned to 0 degrees
- moved IC1 25.7 mm to (233.0, 154.0), turned to 45 degrees
Connections:
- J1 pad 3: Net-(J1-Pad3) -> (no net)
- J1 pad 9: Net-(J1-Pad9) -> (no net)
- R1 pad 2: /CHARGE -> (no net)
- R13 pad 1: Net-(L1-PadA) -> (no net)
- R3 pad 1: Net-(R3-Pad1) -> (no net)
- R6 pad 2: Net-(L2-PadA) -> (no net)
- R7 pad 2: Net-(L3-PadA) -> (no net)
- SW_POW_EN1 pad 3: Net-(SW_POW_EN1-Pad3) -> (no net)
- SW_POW_EN2 pad 3: Net-(SW_POW_EN2-Pad3) -> (no net)
- U1 pad 1: Net-(L4-PadC) -> (no net)
- U2 pad 4: Net-(U2-Pad4) -> (no net)
- U3 pad 10: Net-(U3-Pad10) -> (no net)
- U3 pad 11: Net-(U3-Pad11) -> (no net)
- U3 pad 12: Net-(U3-Pad12) -> (no net)
- U3 pad 15: DCC -> (no net)
- U3 pad 17: Net-(U3-Pad17) -> (no net)
- U3 pad 18: Net-(U3-Pad18) -> (no net)
- U3 pad 19: Net-(U3-Pad19) -> (no net)
- U3 pad 20: Net-(U3-Pad20) -> (no net)
- U3 pad 21: Net-(U3-Pad21) -> (no net)
- U3 pad 22: Net-(U3-Pad22) -> (no net)
- U3 pad 23: Net-(U3-Pad23) -> (no net)
- U3 pad 24: DFU -> (no net)
- U3 pad 26: Net-(U3-Pad26) -> (no net)
- U3 pad 27: Net-(U3-Pad27) -> (no net)
- U3 pad 28: Net-(U3-Pad28) -> (no net)
- U3 pad 29: Net-(U3-Pad29) -> (no net)
- U3 pad 30: Net-(U3-Pad30) -> (no net)
- U3 pad 31: Net-(U3-Pad31) -> (no net)
- U3 pad 32: Net-(U3-Pad32) -> (no net)
- U3 pad 33: Net-(U3-Pad33) -> (no net)
- U3 pad 37: Net-(U3-Pad37) -> (no net)
- U3 pad 40: Net-(U3-Pad40) -> (no net)
- U3 pad 41: DEC2 -> (no net)
- U3 pad 9: Net-(U3-Pad9) -> (no net)
Routing:
- net /ROW0: track 381.9 -> 0.00 mm, vias 2 -> 0
- net /ROW1: track 350.5 -> 0.00 mm, vias 6 -> 0
- net /ROW2: track 305.6 -> 0.00 mm, vias 6 -> 0
- net /COL10: track 297.7 -> 0.00 mm, vias 1 -> 0
- net /ROW3: track 292.8 -> 0.00 mm, vias 6 -> 0
- net /COL11: track 238.2 -> 0.00 mm, vias 1 -> 0
- net /COL0: track 224.2 -> 0.00 mm, vias 1 -> 0
- net /EN: track 209.2 -> 0.00 mm, vias 8 -> 0
- net /COL1: track 203.7 -> 0.00 mm, vias 1 -> 0
- net /COL9: track 201.2 -> 0.00 mm, vias 1 -> 0
- net /COL2: track 187.0 -> 0.00 mm, vias 1 -> 0
- net /COL8: track 185.3 -> 0.00 mm, vias 1 -> 0
- net /COL3: track 170.3 -> 0.00 mm, vias 1 -> 0
- net /COL7: track 157.6 -> 0.00 mm, vias 1 -> 0
- net GND: track 149.8 -> 0.00 mm, vias 35 -> 0
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- added copper zone on In1.Cu, net +3V3
- added copper zone on In2.Cu, net GND
- removed copper zone on B.Cu, net +3V3
- removed copper zone on B.Cu, net GND
- removed copper zone on F.Cu, net GND
Other:
- board size 285 x 94.6 mm -> 285 x 95.1 mm
- copper layers 2 -> 4
- board text added: "1Ah Battery Hole (51x34x5.9mm)"
- board text added: "Shapeshifter 4060 v2.3"
- board text removed: "Laptreus v2.0"

Commit message: try to move all footprints into library. Need to do symbols still
Parts:
- removed J3: Conn_ARM_JTAG_SWD_10, Connector_PinHeader_1.27mm:PinHeader_2x05_P1.27mm_Vertical
- added U4: ARM-JTAG-SWD, Shapeshifter 4060 Footprints:ARM-JTAG-10-SWD-IDC, F.Cu at (256.5, 161.2)
- BOARD1: footprint Laptreus v2_2 Archive Footprints:60-percent-plus-tofu -> Shapeshifter 4060 Footprints:60_percent_plus_tofu_no_center_holes
- C1, C2, C20, C3, C4, C5, C6, C7: footprint Laptreus v2 Footprints:Capacitor-0805MP -> Shapeshifter 4060 Footprints:Capacitor_0805_MP
- D1, D10, D11, D12, D13, D14, D15, D16, D17, D18, D19, D2, D20, D21, D22, D23, D24, D25, D26, D27, D28, D29, D3, D30, D31, D32, D33, D34, D35, D36, D37, D38, D39, D4, D40, D41, D42, D43, D44, D45, D46, D47, D48, D5, D6, D7, D8, D9: footprint Laptreus v2_2 Archive Footprints:D_SOD-323_With_Adhesive -> Shapeshifter 4060 Footprints:D_SOD-323_With_Test_Points
- D49: footprint Adafruit Feather 32u4 Bluefruit LE:SOD-123 -> Shapeshifter 4060 Footprints:D_SOD-323_With_Test_Points
- F1: footprint Laptreus v2_2 Archive Footprints:Fuse_1812_4532Metric_With_Adhesive -> Shapeshifter 4060 Footprints:Fuse_1812_4532Metric
- FID1, FID2, FID3, FID4: footprint Laptreus v2_2 Archive Footprints:FIDUCIAL -> Shapeshifter 4060 Footprints:FIDUCIAL
- IC1: footprint Laptreus v2_2 Archive Footprints:TQFP-44_10x10mm_P0.8mm -> Shapeshifter 4060 Footprints:TQFP-44_10x10mm_P0.8mm
- J1: footprint Laptreus v2 Footprints:HRO-TYPE-C-31-M-12 -> Shapeshifter 4060 Footprints:HRO-TYPE-C-31-M-12
- J2: footprint Laptreus v2 Footprints:isp_standard -> Shapeshifter 4060 Footprints:ISP_Standard
- JP1, JP2, JP3: footprint Adafruit NeoPixel Ring 12:1X01-CLEANBIG -> Shapeshifter 4060 Footprints:1X01-CLEANBIG
- L1, L2, L3, L4: footprint Laptreus v2_2 Archive Footprints:LED_0603_1608Metric_Castellated_With_Adhesive -> Shapeshifter 4060 Footprints:LED_0603_1608Metric_Castellated
- R1, R10, R11, R12, R13, R2, R3, R4, R5, R6, R7, R8, R9: footprint Laptreus v2_2 Archive Footprints:R_0603_1608Metric_With_Adhesive -> Shapeshifter 4060 Footprints:R_0603_1608Metric
- S9: footprint Laptreus v2 Footprints:PKRH -> Shapeshifter 4060 Footprints:5mm_M2.5_Screw_Hole_Plated
- SW1, SW10, SW11, SW12, SW13, SW15, SW16, SW17, SW18, SW19, SW2, SW20, SW21, SW22, SW26, SW27, SW28, SW29, SW3, SW30, SW31, SW32, SW33, SW34, SW35, SW37, SW38, SW39, SW4, SW40, SW41, SW42, SW43, SW44, SW45, SW46, SW47, SW48, SW5, SW6, SW7, SW8, SW9: footprint Laptreus v2_2 Archive Footprints:Hybrid_Kailh_MX_Choc_Socket_Through_Hole_With_Diode -> Shapeshifter 4060 Footprints:Kailh_Socket_With_Diode
- SW14, SW23, SW24, SW25, SW36: footprint Laptreus v2_2 Archive Footprints:Hybrid_Kailh_MX_Choc_Socket_Through_Hole_With_Diode_No_Diode_Trace -> Shapeshifter 4060 Footprints:Kailh_Socket_With_Diode
- SW_POW_EN1, SW_POW_EN2: footprint Laptreus v2 Footprints:EG1218 -> Shapeshifter 4060 Footprints:EG1218
- SW_RESET1: footprint Laptreus v2 Footprints:SW_SPST_B3U-1000P -> Shapeshifter 4060 Footprints:SW_SPST_B3U-1000P
- U1, U2: footprint Laptreus v2_2 Archive Footprints:SOT-143_With_Adhesive -> Shapeshifter 4060 Footprints:SOT-23-5
- U3: footprint Adafruit Feather 32u4 Bluefruit LE:BLE_MODULE_RAYTAC_MDBT40 -> Shapeshifter 4060 Footprints:BLE_MODULE_RAYTAC_MDBT40
- U6: footprint Laptreus v2 Footprints:USBLC6-2SC6 -> Shapeshifter 4060 Footprints:SOT-23-6
- X1, X2: footprint Laptreus v2_2 Archive Footprints:JSTPH2-with-THT -> Shapeshifter 4060 Footprints:JSTPH2_With_THT
- Y1: footprint Adafruit Feather 32u4 Bluefruit LE:RESONATOR-SMD -> Shapeshifter 4060 Footprints:3_Pin_SMD_Resonator
- moved L1 153.5 mm to (248.0, 158.5), turned to 270 degrees
- moved R13 152.5 mm to (246.5, 158.5), turned to 270 degrees
- moved L2 150.5 mm to (245.0, 158.5), turned to 270 degrees
- moved R6 149.6 mm to (243.5, 158.5), turned to 270 degrees
- moved U3 129.0 mm to (232.8, 157.0)
- moved R1 128.4 mm to (222.5, 158.5), turned to 270 degrees
- moved L4 126.5 mm to (221.0, 158.5), turned to 270 degrees
- moved R7 126.0 mm to (219.5, 158.5), turned to 270 degrees
- moved L3 123.7 mm to (218.0, 158.5), turned to 270 degrees
- moved C2 79.6 mm to (225.0, 158.5), turned to 270 degrees
- moved J2 25.4 mm to (221.5, 133.5)
- moved IC1 16.5 mm to (233.2, 137.5)
Connections:
- D1 pad 1: Net-(D1-Pad1) -> /COL11
- D1 pad 2: /COL11 -> Net-(D1-Pad2)
- D10 pad 1: Net-(D10-Pad1) -> /COL2
- D10 pad 2: /COL2 -> Net-(D10-Pad2)
- D11 pad 1: Net-(D11-Pad1) -> /COL1
- D11 pad 2: /COL1 -> Net-(D11-Pad2)
- D12 pad 1: Net-(D12-Pad1) -> /COL0
- D12 pad 2: /COL0 -> Net-(D12-Pad2)
- D13 pad 1: Net-(D13-Pad1) -> /COL11
- D13 pad 2: /COL11 -> Net-(D13-Pad2)
- D14 pad 1: Net-(D14-Pad1) -> /COL10
- D14 pad 2: /COL10 -> Net-(D14-Pad2)
- D15 pad 1: Net-(D15-Pad1) -> /COL9
- D15 pad 2: /COL9 -> Net-(D15-Pad2)
- D16 pad 1: Net-(D16-Pad1) -> /COL8
- D16 pad 2: /COL8 -> Net-(D16-Pad2)
- D17 pad 1: Net-(D17-Pad1) -> /COL7
- D17 pad 2: /COL7 -> Net-(D17-Pad2)
- D18 pad 1: Net-(D18-Pad1) -> /COL6
- D18 pad 2: /COL6 -> Net-(D18-Pad2)
- D19 pad 1: Net-(D19-Pad1) -> /COL5
- D19 pad 2: /COL5 -> Net-(D19-Pad2)
- D2 pad 1: Net-(D2-Pad1) -> /COL10
- D2 pad 2: /COL10 -> Net-(D2-Pad2)
- D20 pad 1: Net-(D20-Pad1) -> /COL4
- D20 pad 2: /COL4 -> Net-(D20-Pad2)
- D21 pad 1: Net-(D21-Pad1) -> /COL3
- D21 pad 2: /COL3 -> Net-(D21-Pad2)
- D22 pad 1: Net-(D22-Pad1) -> /COL2
- D22 pad 2: /COL2 -> Net-(D22-Pad2)
- D23 pad 1: Net-(D23-Pad1) -> /COL1
- D23 pad 2: /COL1 -> Net-(D23-Pad2)
- D24 pad 1: Net-(D24-Pad1) -> /COL0
- D24 pad 2: /COL0 -> Net-(D24-Pad2)
- D25 pad 1: Net-(D25-Pad1) -> /COL11
- D25 pad 2: /COL11 -> Net-(D25-Pad2)
- D26 pad 1: Net-(D26-Pad1) -> /COL10
- D26 pad 2: /COL10 -> Net-(D26-Pad2)
- D27 pad 1: Net-(D27-Pad1) -> /COL9
- D27 pad 2: /COL9 -> Net-(D27-Pad2)
- D28 pad 1: Net-(D28-Pad1) -> /COL8
- D28 pad 2: /COL8 -> Net-(D28-Pad2)
- D29 pad 1: Net-(D29-Pad1) -> /COL7
- D29 pad 2: /COL7 -> Net-(D29-Pad2)
- D3 pad 1: Net-(D3-Pad1) -> /COL9
- D3 pad 2: /COL9 -> Net-(D3-Pad2)
- D30 pad 1: Net-(D30-Pad1) -> /COL6
- D30 pad 2: /COL6 -> Net-(D30-Pad2)
- D31 pad 1: Net-(D31-Pad1) -> /COL5
- D31 pad 2: /COL5 -> Net-(D31-Pad2)
- D32 pad 1: Net-(D32-Pad1) -> /COL4
- D32 pad 2: /COL4 -> Net-(D32-Pad2)
- D33 pad 1: Net-(D33-Pad1) -> /COL3
- D33 pad 2: /COL3 -> Net-(D33-Pad2)
- D34 pad 1: Net-(D34-Pad1) -> /COL2
- D34 pad 2: /COL2 -> Net-(D34-Pad2)
- D35 pad 1: Net-(D35-Pad1) -> /COL1
- D35 pad 2: /COL1 -> Net-(D35-Pad2)
- D36 pad 1: Net-(D36-Pad1) -> /COL0
- D36 pad 2: /COL0 -> Net-(D36-Pad2)
- D37 pad 1: Net-(D37-Pad1) -> /COL11
- D37 pad 2: /COL11 -> Net-(D37-Pad2)
- D38 pad 1: Net-(D38-Pad1) -> /COL10
- D38 pad 2: /COL10 -> Net-(D38-Pad2)
- D39 pad 1: Net-(D39-Pad1) -> /COL9
- D39 pad 2: /COL9 -> Net-(D39-Pad2)
- D4 pad 1: Net-(D4-Pad1) -> /COL8
- D4 pad 2: /COL8 -> Net-(D4-Pad2)
- D40 pad 1: Net-(D40-Pad1) -> /COL8
- D40 pad 2: /COL8 -> Net-(D40-Pad2)
- D41 pad 1: Net-(D41-Pad1) -> /COL7
- D41 pad 2: /COL7 -> Net-(D41-Pad2)
- D42 pad 1: Net-(D42-Pad1) -> /COL6
- D42 pad 2: /COL6 -> Net-(D42-Pad2)
- D43 pad 1: Net-(D43-Pad1) -> /COL5
- D43 pad 2: /COL5 -> Net-(D43-Pad2)
- D44 pad 1: Net-(D44-Pad1) -> /COL4
- D44 pad 2: /COL4 -> Net-(D44-Pad2)
- D45 pad 1: Net-(D45-Pad1) -> /COL3
- D45 pad 2: /COL3 -> Net-(D45-Pad2)
- D46 pad 1: Net-(D46-Pad1) -> /COL2
- D46 pad 2: /COL2 -> Net-(D46-Pad2)
- D47 pad 1: Net-(D47-Pad1) -> /COL1
- D47 pad 2: /COL1 -> Net-(D47-Pad2)
- D48 pad 1: Net-(D48-Pad1) -> /COL0
- D48 pad 2: /COL0 -> Net-(D48-Pad2)
- D5 pad 1: Net-(D5-Pad1) -> /COL7
- D5 pad 2: /COL7 -> Net-(D5-Pad2)
- D6 pad 1: Net-(D6-Pad1) -> /COL6
- D6 pad 2: /COL6 -> Net-(D6-Pad2)
- D7 pad 1: Net-(D7-Pad1) -> /COL5
- D7 pad 2: /COL5 -> Net-(D7-Pad2)
- D8 pad 1: Net-(D8-Pad1) -> /COL4
- D8 pad 2: /COL4 -> Net-(D8-Pad2)
- D9 pad 1: Net-(D9-Pad1) -> /COL3
- D9 pad 2: /COL3 -> Net-(D9-Pad2)
- R1 pad 1: +5V -> /CHARGE
- R1 pad 2: (no net) -> +5V
- R13 pad 1: (no net) -> Net-(L1-PadA)
- R3 pad 1: (no net) -> Net-(R3-Pad1)
- R6 pad 1: /MODE -> Net-(L2-PadA)
- R6 pad 2: (no net) -> /MODE
- R7 pad 1: /CONNECTED -> Net-(L3-PadA)
- R7 pad 2: (no net) -> /CONNECTED
- SW1 pad 2: Net-(D1-Pad1) -> Net-(D1-Pad2)
- SW10 pad 2: Net-(D10-Pad1) -> Net-(D10-Pad2)
- SW11 pad 2: Net-(D11-Pad1) -> Net-(D11-Pad2)
- SW12 pad 2: Net-(D12-Pad1) -> Net-(D12-Pad2)
- SW13 pad 2: Net-(D13-Pad1) -> Net-(D13-Pad2)
- SW14 pad 2: Net-(D14-Pad1) -> Net-(D14-Pad2)
- SW15 pad 2: Net-(D15-Pad1) -> Net-(D15-Pad2)
- SW16 pad 2: Net-(D16-Pad1) -> Net-(D16-Pad2)
- SW17 pad 2: Net-(D17-Pad1) -> Net-(D17-Pad2)
- SW18 pad 2: Net-(D18-Pad1) -> Net-(D18-Pad2)
- SW19 pad 2: Net-(D19-Pad1) -> Net-(D19-Pad2)
- SW2 pad 2: Net-(D2-Pad1) -> Net-(D2-Pad2)
- SW20 pad 2: Net-(D20-Pad1) -> Net-(D20-Pad2)
- SW21 pad 2: Net-(D21-Pad1) -> Net-(D21-Pad2)
- SW22 pad 2: Net-(D22-Pad1) -> Net-(D22-Pad2)
- SW23 pad 2: Net-(D23-Pad1) -> Net-(D23-Pad2)
- SW24 pad 2: Net-(D24-Pad1) -> Net-(D24-Pad2)
- SW25 pad 2: Net-(D25-Pad1) -> Net-(D25-Pad2)
- SW26 pad 2: Net-(D26-Pad1) -> Net-(D26-Pad2)
- SW27 pad 2: Net-(D27-Pad1) -> Net-(D27-Pad2)
- SW28 pad 2: Net-(D28-Pad1) -> Net-(D28-Pad2)
- SW29 pad 2: Net-(D29-Pad1) -> Net-(D29-Pad2)
- SW3 pad 2: Net-(D3-Pad1) -> Net-(D3-Pad2)
- SW30 pad 2: Net-(D30-Pad1) -> Net-(D30-Pad2)
- SW31 pad 2: Net-(D31-Pad1) -> Net-(D31-Pad2)
- SW32 pad 2: Net-(D32-Pad1) -> Net-(D32-Pad2)
- SW33 pad 2: Net-(D33-Pad1) -> Net-(D33-Pad2)
- SW34 pad 2: Net-(D34-Pad1) -> Net-(D34-Pad2)
- SW35 pad 2: Net-(D35-Pad1) -> Net-(D35-Pad2)
- SW36 pad 2: Net-(D36-Pad1) -> Net-(D36-Pad2)
- SW37 pad 2: Net-(D37-Pad1) -> Net-(D37-Pad2)
- SW38 pad 2: Net-(D38-Pad1) -> Net-(D38-Pad2)
- SW39 pad 2: Net-(D39-Pad1) -> Net-(D39-Pad2)
- SW4 pad 2: Net-(D4-Pad1) -> Net-(D4-Pad2)
- SW40 pad 2: Net-(D40-Pad1) -> Net-(D40-Pad2)
- SW41 pad 2: Net-(D41-Pad1) -> Net-(D41-Pad2)
- SW42 pad 2: Net-(D42-Pad1) -> Net-(D42-Pad2)
- SW43 pad 2: Net-(D43-Pad1) -> Net-(D43-Pad2)
- SW44 pad 2: Net-(D44-Pad1) -> Net-(D44-Pad2)
- SW45 pad 2: Net-(D45-Pad1) -> Net-(D45-Pad2)
- SW46 pad 2: Net-(D46-Pad1) -> Net-(D46-Pad2)
- SW47 pad 2: Net-(D47-Pad1) -> Net-(D47-Pad2)
- SW48 pad 2: Net-(D48-Pad1) -> Net-(D48-Pad2)
- SW5 pad 2: Net-(D5-Pad1) -> Net-(D5-Pad2)
- SW6 pad 2: Net-(D6-Pad1) -> Net-(D6-Pad2)
- SW7 pad 2: Net-(D7-Pad1) -> Net-(D7-Pad2)
- SW8 pad 2: Net-(D8-Pad1) -> Net-(D8-Pad2)
- SW9 pad 2: Net-(D9-Pad1) -> Net-(D9-Pad2)
- U1 pad 1: (no net) -> Net-(L4-PadC)
Routing:
- removed copper zone on F.Cu, net (none)
