File: pcb/Shapeshifter_4060_v3/kicad/Laptreus-v3.sch (KiCad schematic (older format))
At the start: 111 parts, among them SW1 TAB, SW10 O, SW11 P, SW12 BKSP, SW13 ESC, SW14 A, SW15 S, SW16 D, SW17 F, SW18 G, SW19 H, SW2 Q, SW20 J, SW21 K, SW22 L, SW23 ;, SW24 ENTER, SW25 SHIFT, SW26 Z, SW27 X, SW28 C, SW29 V, SW3 W, SW30 B, SW31 N, SW32 M, SW33 ,, SW34 ., SW35 /, SW36 SHIFT, SW37 CTRL/ESC, SW38 ALT/GRV, SW39 CMD, SW4 E, SW40 FN1, SW41 SHIFT, SW42 BKSP, SW43 ENTER, SW44 SPACE, SW45 LEFT, SW46 DOWN, SW47 UP, SW48 RIGHT, SW5 R, SW6 T, SW7 Y, SW8 U, SW9 I, U1 nice_nano

Commit message: Add BOM/pos files for pcba
Parts:
- BOARD1, FID1, FID2, FID3, FID4, FID5, FID6, JP1, JP2, JP3, JP4, JP5, JP6, U1: Vendor (none) -> N/A
- D1, D10, D11, D12, D13, D14, D15, D16, D17, D18, D19, D2, D20, D21, D22, D23, D24, D25, D26, D27, D28, D29, D3, D30, D31, D32, D33, D34, D35, D36, D37, D38, D39, D4, D40, D41, D42, D43, D44, D45, D46, D47, D48, D5, D6, D7, D8, D9: Designation (none) -> SOD-123 2L; Vendor (none) -> MMSD4148
- SW1, SW10, SW11, SW12, SW13, SW14, SW15, SW16, SW17, SW18, SW19, SW2, SW20, SW21, SW22, SW23, SW24, SW25, SW26, SW27, SW28, SW29, SW3, SW30, SW31, SW32, SW33, SW34, SW35, SW36, SW37, SW38, SW39, SW4, SW40, SW41, SW42, SW43, SW44, SW45, SW46, SW47, SW48, SW5, SW6, SW7, SW8, SW9: Vendor (none) -> CPG151101S11
- SW_RESET_1: Vendor (none) -> B3U-1000P-2P-SMD
